Commit message: adding Map My World

File: src/my_robot/urdf/my_robot.xacro (robot description, xacro)
@@ -175,5 +175,12 @@
     <axis xyz="0 1 0" rpy="0 0 0"/>
   </joint>
-  <!-- ******* -->
+  <!-- camera optical joint -->
+  <joint name="camera_optical_joint" type="fixed">
+    <origin xyz="0 0 0" rpy="-1.5707 0 -1.5707"/>
+    <parent link="camera_link"/>
+    <child link="camera_link_optical"/>
+  </joint>
+  <link name="camera_link_optical">
+  </link>
   <!-- ******* LIDAR ******* -->
   <link name="hokuyo">

Commit message: fix camera_link to camera

File: src/my_robot/urdf/my_robot.xacro (robot description, xacro)
@@ -178,6 +178,6 @@
   <joint name="camera_optical_joint" type="fixed">
     <origin xyz="0 0 0" rpy="-1.5707 0 -1.5707"/>
-    <parent link="camera_link"/>
-    <child link="camera_link_optical"/>
+    <parent link="camera"/>
+    <child link="camera_optical"/>
   </joint>
   <link name="camera_link_optical">

Commit message: fix camera_link to camera

File: src/my_robot/urdf/my_robot.xacro (robot description, xacro)
@@ -181,5 +181,6 @@
     <child link="camera_optical"/>
   </joint>
-  <link name="camera_link_optical">
+<!-- Camera Optical Link -->
+ <link name="camera_optical">
   </link>
   <!-- ******* LIDAR ******* -->
